Commit message: test

File: un_robot/ur_description/urdf/ur3.urdf.xacro (robot description, xacro)
@@ -229,5 +229,4 @@
       </inertial>
     </link>
-<!--
      <joint name="${prefix}ur3_mount_joint" type="revolute">
       <parent link="${prefix}ur3_mount" />
@@ -266,6 +265,6 @@
         <origin xyz="0.0 0.0 0.0" rpy="0 0 0" />
       </xacro:cylinder_inertial>
-    </link> -->
-    <!-- <joint name="${prefix}shoulder_pan_joint" type="revolute">
+    </link>
+    <joint name="${prefix}shoulder_pan_joint" type="revolute">
       <parent link="${prefix}bottom_link" />
       <child link = "${prefix}shoulder_link" />
@@ -501,5 +500,5 @@
         <origin rpy="0 0 0" xyz="-0.01 0 0"/>
       </collision>
-    </link>  -->
+    </link>
     <xacro:ur_arm_transmission prefix="${prefix}" hw_interface="${transmission_hw_interface}" />
     <xacro:ur_arm_gazebo prefix="${prefix}" />
