Commit message: last bug fixes

File: Suii/suii_description/Field/rack_bin/urdf/rack_bin_blue.urdf (robot description, URDF)
Before this commit: robot rack_bin, 1 links, 0 joints
Links:
- link rack_bin: geometry collision mesh filename=package://suii_description/Field/rack_bin/meshes/blue_bin.d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; visual mesh filename=package://suii_description/Field/rack_bin/meshes/blue_bin.d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

File: Suii/suii_description/Field/rack_bin/urdf/rack_bin_red.urdf (robot description, URDF)
Before this commit: robot rack_bin, 1 links, 0 joints
Links:
- link rack_bin: geometry collision mesh filename=package://suii_description/Field/rack_bin/meshes/red_bin.dae; visual mesh filename=package://suii_description/Field/rack_bin/meshes/red_bin.dae
