Commit message: table movement fix

File: Suii/suii_description/Field/objects/urdf/alu_prof_large_black.urdf (robot description, URDF)
Before this commit: robot Part2.SLDPRT, 1 links, 0 joints
Links:
- removed link Extrusion_40x40.SLDPRT
- added link alu_prof_large_black, mass 0.186; collision mesh filename=package://suii_description/Field/objects/meshes/alu_prof_la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; visual mesh filename=package://suii_description/Field/objects/meshes/alu_prof_la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

File: Suii/suii_description/Field/objects/urdf/alu_prof_large_gray.urdf (robot description, URDF)
Before this commit: robot Part2.SLDPRT, 1 links, 0 joints
Links:
- removed link Extrusion_40x40.SLDPRT
- added link alu_prof_large_gray, mass 0.186; collision mesh filename=package://suii_description/Field/objects/meshes/alu_prof_la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; visual mesh filename=package://suii_description/Field/objects/meshes/alu_prof_la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
