Commit message: gripper added

File: Suii/suii_description/urdf/suii.xacro (robot description, xacro)
@@ -514,7 +514,49 @@
         </geometry>
       </collision>
-      <xacro:cylinder_inertial radius="0.032" length="0.04" mass="${wrist_3_mass}">
-        <origin xyz="0.0 ${wrist_3_length - 0.02} 0.0" rpy="${pi/2} 0 0" />
-      </xacro:cylinder_inertial>
+      <inertial>
+        <mass value= "${frame_mass}"/>
+        <inertia ixx="0.0" ixy="0.0" ixz="0.0" iyy="0" iyz="0" izz="0"/>
+        <origin xyz="0 0 0"  rpy="0 0 0" />
+      </inertial>
+    </link>
+<!--  -->
+    <joint name="${prefix}servo_link" type="fixed">
+      <parent link="${prefix}base_gripper" />
+      <child link = "${prefix}servo_link" />
+      <origin xyz="0.0 0.1 0.0" rpy="1.57 1.57 0" />
+      <axis xyz="0 1 0" />
+      <!-- <xacro:unless value="${joint_limited}">
+        <limit lower="${-2.0 * pi}" upper="${2.0 * pi}" effort="54.0" velocity="3.2"/>
+        <xacro:if value="${safety_limits}">
+          <safety_controller soft_lower_limit="${-2.0 * pi + safety_pos_margin}" soft_upper_limit="${2.0 * pi - safety_pos_margin}" k_position="${safety_k_position}" k_velocity="0.0"/>
+        </xacro:if>
+      </xacro:unless>
+      <xacro:if value="${joint_limited}">
+        <limit lower="${wrist_3_lower_limit}" upper="${wrist_3_upper_limit}" effort="54.0" velocity="3.2"/>
+        <xacro:if value="${safety_limits}">
+          <safety_controller soft_lower_limit="${wrist_3_lower_limit + safety_pos_margin}" soft_upper_limit="${wrist_3_upper_limit - safety_pos_margin}" k_position="${safety_k_position}" k_velocity="0.0"/>
+        </xacro:if>
+      </xacro:if>
+      <dynamics damping="0.0" friction="0.0"/> -->
+    </joint>
+    <link name="${prefix}servo_link">
+      <visual>
+        <geometry>
+          <mesh filename="package://suii_description/meshes/suii/visual/servo_link.stl"/>
+        </geometry>
+        <material name="LightGrey">
+          <color rgba="0.7 0.7 0.7 1.0"/>
+        </material>
+      </visual>
+      <collision>
+        <geometry>
+          <mesh filename="package://suii_description/meshes/suii/collision/servo_link.stl"/>
+        </geometry>
+      </collision>
+      <inertial>
+        <mass value= "${frame_mass}"/>
+        <inertia ixx="0.0" ixy="0.0" ixz="0.0" iyy="0" iyz="0" izz="0"/>
+        <origin xyz="0 0 0"  rpy="0 0 0" />
+      </inertial>
     </link>
     <!-- <link name="${prefix}ee_link">

File: Suii_Gripper/urdf/gripper.urdf (robot description, URDF)
Before this commit: robot gripper, 8 links, 7 joints
Links:
- removed link base_link

Commit message: add sensors on Suii

File: Suii/suii_description/urdf/suii.xacro (robot description, xacro)
@@ -57,4 +57,9 @@
     <xacro:property name="wrist_2_length" value="${d5}" />
     <xacro:property name="wrist_3_length" value="${d6}" />
+    <!-- sensor properties-->
+    <xacro:property name="sonar_link" value="-0.05" /> <!-- Size of square 'sonar' box -->
+    <xacro:property name="laser_link" value="-0.05" /> <!-- Size of square 'sonar' box -->
+    <xacro:property name="height" value="0.3" /> <!-- height sensors-->
+    <xacro:property name="axel_offset" value="0.05" /> <!-- offset placement -->
     <gazebo>
 	    <plugin name="omni_steering" filename="libgazebo_ros_planar_move.so">
@@ -489,4 +494,60 @@
       </collision>
     </link>
+    <!-- sonar -->
+    <link name="sonar_link">
+      <collision>
+        <origin xyz="0 0 0" rpy="0 0 0"/>
+        <geometry>
+          <box size="${sonar_link} ${sonar_link} ${sonar_link}"/>
+        </geometry>
+      </collision>
+      <visual>
+        <origin xyz="0 0 0" rpy="0 0 0"/>
+        <geometry>
+          <box size="${sonar_link} ${sonar_link} ${sonar_link}"/>
+        </geometry>
+        <material name="blue"/>
+      </visual>
+      <inertial>
+        <mass value="1e-5" />
+        <origin xyz="0 0 0" rpy="0 0 0"/>
+        <inertia ixx="1e-6" ixy="0" ixz="0" iyy="1e-6" iyz="0" izz="1e-6" />
+      </inertial>
+    </link>
+    <!-- sonar joint -->
+    <joint name="sonar_joint" type="fixed">
+      <axis xyz= "0 1 0" />
+      <origin xyz="-0.275 0 0.1" rpy="0 0 3.1415926535897931"/>
+      <parent link="${prefix}base_link"/>
+      <child link="sonar_link"/>
+    </joint>
+    <!-- Hokuyo Laser -->
+    <link name="hokuyo_link">
+      <collision>
+        <origin xyz="0 0 0" rpy="0 0 0"/>
+        <geometry>
+          <box size="0.1 0.1 0.1"/>
+        </geometry>
+      </collision>
+      <visual>
+        <origin xyz="0 0 0" rpy="0 0 0"/>
+        <geometry>
+          <box size="${laser_link} ${laser_link} ${laser_link}"/>
+        </geometry>
+        <material name="red"/>
+      </visual>
+      <inertial>
+        <mass value="1e-5" />
+        <origin xyz="0 0 0" rpy="0 0 0"/>
+        <inertia ixx="1e-6" ixy="0" ixz="0" iyy="1e-6" iyz="0" izz="1e-6" />
+      </inertial>
+    </link>
+    <!-- laser joint -->
+    <joint name="hokuyo_joint" type="fixed">
+      <axis xyz="0 1 0" />
+      <origin xyz="0.035 0 0.25" rpy="0 0 0"/>
+      <parent link="${prefix}base_link"/>
+      <child link="hokuyo_link"/>
+    </joint>
     <xacro:suii_transmission prefix="${prefix}" hw_interface="${transmission_hw_interface}" />
     <xacro:suii_gazebo prefix="${prefix}" />

File: Suii/suii_description/urdf/suii_gazebo.xacro (robot description, xacro)
@@ -93,4 +93,74 @@
       <selfCollide>true</selfCollide>
     </gazebo>
+    <!-- hokuyo -->
+    <gazebo reference="hokuyo_link">
+      <sensor type="gpu_ray" name="head_hokuyo_sensor">
+        <pose>0 0 0 0 0 0</pose>
+        <visualize>false</visualize>
+        <update_rate>40</update_rate>
+        <ray>
+          <scan>
+            <horizontal>
+              <samples>720</samples>
+              <resolution>1</resolution>
+              <min_angle>-1.570796</min_angle>
+              <max_angle>1.570796</max_angle>
+            </horizontal>
+          </scan>
+          <range>
+            <min>0.10</min>
+            <max>30.0</max>
+            <resolution>0.01</resolution>
+          </range>
+          <noise>
+            <type>gaussian</type>
+            <mean>0.0</mean>
+            <stddev>0.01</stddev>
+          </noise>
+        </ray>
+        <plugin name="gazebo_ros_head_hokuyo_controller" filename="libgazebo_ros_gpu_laser.so">
+          <topicName>/suii/laser/scan</topicName>
+          <frameName>hokuyo_link</frameName>
+        </plugin>
+      </sensor>
+    </gazebo>
+    <!-- sonar -->
+    <gazebo reference="sonar_link">
+      <sensor type="ray" name="sonar_sensor">
+        <pose>0 0 0 0 0 0</pose>
+        <update_rate>50</update_rate>
+        <ray>
+          <scan>
+              <horizontal>
+                <samples>10</samples>
+                <resolution>1.0</resolution>
+                <min_angle>-0.01</min_angle>
+                <max_angle>0.01</max_angle>
+              </horizontal>
+              <vertical>
+                <samples>10</samples>
+                <resolution>1</resolution>
+                <min_angle>-0.01</min_angle>
+                <max_angle>0.01</max_angle>
+              </vertical>
+          </scan>
+          <range>
+              <min>0.01</min>
+              <max>3.75</max>
+              <resolution>0.02</resolution>
+          </range>
+        </ray>
+        <plugin filename="libgazebo_ros_range.so" name="gazebo_ros_range">
+          <gaussianNoise>0.005</gaussianNoise>
+          <alwaysOn>true</alwaysOn>
+          <updateRate>5</updateRate>
+          <topicName>/suii/sonar/scan</topicName>
+          <frameName>sonar_link</frameName>
+          <visualize>true</visualize>
+          <radiation>infrared</radiation>
+          <fov>0.2</fov>
+        </plugin>
+      </sensor>
+    </gazebo>
   </xacro:macro>
 </robot>

File: ros_senors_gazebo/rrbot_description/urdf/rrbot.xacro (robot description, xacro)
@@ -106,5 +106,5 @@
 	  iyy="${mass / 12.0 * (height3*height3 + width*width)}" iyz="0.0"
 	  izz="${mass / 12.0 * (width*width + width*width)}"/>
-    </inertial>sonar_link
+    </inertial>
   </link>
   <joint name="sonar_joint" type="fixed">

File: sensor_mount_test/ur_description/urdf/mybot_gazebo_plugins.xacro (robot description, xacro)
@@ -55,2 +55,40 @@
   </sensor>
 </gazebo>
+<!-- sonar -->
+<gazebo reference="sonar_link">
+  <sensor type="ray" name="sonar_sensor">
+    <pose>0 0 0 0 0 0</pose>
+    <update_rate>50</update_rate>
+    <ray>
+        <scan>
+          <horizontal>
+              <samples>10</samples>
+              <resolution>1.0</resolution>
+              <min_angle>-0.01</min_angle>
+              <max_angle>0.01</max_angle>
+          </horizontal>
+          <vertical>
+              <samples>10</samples>
+              <resolution>1</resolution>
+              <min_angle>-0.01</min_angle>
+              <max_angle>0.01</max_angle>
+          </vertical>
+        </scan>
+        <range>
+          <min>0.01</min>
+          <max>3.75</max>
+          <resolution>0.02</resolution>
+        </range>
+    </ray>
+    <plugin filename="libgazebo_ros_range.so" name="gazebo_ros_range">
+        <gaussianNoise>0.005</gaussianNoise>
+        <alwaysOn>true</alwaysOn>
+        <updateRate>5</updateRate>
+        <topicName>/suii/sonar/scan</topicName>
+        <frameName>sonar_link</frameName>
+        <visualize>true</visualize>
+        <radiation>infrared</radiation>
+        <fov>0.2</fov>
+    </plugin>
+  </sensor>
+</gazebo>

File: sensor_mount_test/ur_description/urdf/ur.gazebo.xacro (robot description, xacro)
@@ -8,5 +8,5 @@
       <selfCollide>true</selfCollide>
     </gazebo>
-    <!-- <gazebo reference="${prefix}left_front_wheel_link">
+    <gazebo reference="${prefix}left_front_wheel_link">
       <selfCollide>true</selfCollide>
     </gazebo>
@@ -18,6 +18,6 @@
     </gazebo>
     <gazebo reference="${prefix}right_back_wheel_link">
-      <selfCollide>true</selfCollide> -->
-    <!-- </gazebo> -->
+      <selfCollide>true</selfCollide>
+    </gazebo>
     <gazebo reference="${prefix}bottum_link">
       <selfCollide>true</selfCollide>
@@ -44,4 +44,73 @@
       <selfCollide>true</selfCollide>
     </gazebo>
+    <gazebo reference="hokuyo_link">
+      <sensor type="gpu_ray" name="head_hokuyo_sensor">
+        <pose>0 0 0 0 0 0</pose>
+        <visualize>false</visualize>
+        <update_rate>40</update_rate>
+        <ray>
+          <scan>
+            <horizontal>
+              <samples>720</samples>
+              <resolution>1</resolution>
+              <min_angle>-1.570796</min_angle>
+              <max_angle>1.570796</max_angle>
+            </horizontal>
+          </scan>
+          <range>
+            <min>0.10</min>
+            <max>30.0</max>
+            <resolution>0.01</resolution>
+          </range>
+          <noise>
+            <type>gaussian</type>
+            <mean>0.0</mean>
+            <stddev>0.01</stddev>
+          </noise>
+        </ray>
+        <plugin name="gazebo_ros_head_hokuyo_controller" filename="libgazebo_ros_gpu_laser.so">
+          <topicName>/suii/laser/scan</topicName>
+          <frameName>hokuyo_link</frameName>
+        </plugin>
+      </sensor>
+    </gazebo>
+    <!-- sonar -->
+    <gazebo reference="sonar_link">
+      <sensor type="ray" name="sonar_sensor">
+        <pose>0 0 0 0 0 0</pose>
+        <update_rate>50</update_rate>
+        <ray>
+            <scan>
+              <horizontal>
+                  <samples>10</samples>
+                  <resolution>1.0</resolution>
+                  <min_angle>-0.01</min_angle>
+                  <max_angle>0.01</max_angle>
+              </horizontal>
+              <vertical>
+                  <samples>10</samples>
+                  <resolution>1</resolution>
+                  <min_angle>-0.01</min_angle>
+                  <max_angle>0.01</max_angle>
+              </vertical>
+            </scan>
+            <range>
+              <min>0.01</min>
+              <max>3.75</max>
+              <resolution>0.02</resolution>
+            </range>
+        </ray>
+        <plugin filename="libgazebo_ros_range.so" name="gazebo_ros_range">
+            <gaussianNoise>0.005</gaussianNoise>
+            <alwaysOn>true</alwaysOn>
+            <updateRate>5</updateRate>
+            <topicName>/suii/sonar/scan</topicName>
+            <frameName>sonar_link</frameName>
+            <visualize>true</visualize>
+            <radiation>infrared</radiation>
+            <fov>0.2</fov>
+        </plugin>
+      </sensor>
+    </gazebo>
   </xacro:macro>
 </robot>

File: sensor_mount_test/ur_description/urdf/ur3.urdf.xacro (robot description, xacro)
@@ -102,63 +102,59 @@
       <axis xyz="0 0 1" />
     </joint>
-    <!-- hokuyo -->
-    <gazebo reference="hokuyo_link">
-      <sensor type="gpu_ray" name="head_hokuyo_sensor">
-        <pose>0 0 0 0 0 0</pose>
-        <visualize>false</visualize>
-        <update_rate>40</update_rate>
-        <ray>
-          <scan>
-            <horizontal>
-              <samples>720</samples>
-              <resolution>1</resolution>
-              <min_angle>-1.570796</min_angle>
-              <max_angle>1.570796</max_angle>
-            </horizontal>
-          </scan>
-          <range>
-            <min>0.10</min>
-            <max>30.0</max>
-            <resolution>0.01</resolution>
-          </range>
-          <noise>
-            <type>gaussian</type>
-            <mean>0.0</mean>
-            <stddev>0.01</stddev>
-          </noise>
-        </ray>
-        <plugin name="gazebo_ros_head_hokuyo_controller" filename="libgazebo_ros_gpu_laser.so">
-          <topicName>/suii/laser/scan</topicName>
-          <frameName>hokuyo_link</frameName>
-        </plugin>
-      </sensor>
-    </gazebo>
-    <!-- laser-->
+    <!-- sonar -->
+    <link name="sonar_link">
+      <collision>
+        <origin xyz="0 0 0" rpy="0 0 0"/>
+        <geometry>
+          <box size="${sonar_link} ${sonar_link} ${sonar_link}"/>
+        </geometry>
+      </collision>
+      <visual>
+        <origin xyz="0 0 0" rpy="0 0 0"/>
+        <geometry>
+          <box size="${sonar_link} ${sonar_link} ${sonar_link}"/>
+        </geometry>
+        <material name="blue"/>
+      </visual>
+      <inertial>
+        <mass value="1e-5" />
+        <origin xyz="0 0 0" rpy="0 0 0"/>
+        <inertia ixx="1e-6" ixy="0" ixz="0" iyy="1e-6" iyz="0" izz="1e-6" />
+      </inertial>
+    </link>
+    <!-- sonar joint -->
+    <joint name="sonar_joint" type="fixed">
+      <axis xyz= "0 1 0" />
+      <origin xyz="${sonar_link} 0 ${height3 - axel_offset*2}" rpy="0 0 3.1415926535897931"/>
+      <parent link="${prefix}base_link"/>
+      <child link="sonar_link"/>
+    </joint>
+    <!-- Hokuyo Laser -->
+    <link name="hokuyo_link">
+      <collision>
+        <origin xyz="0 0 0" rpy="0 0 0"/>
+        <geometry>
+          <box size="0.1 0.1 0.1"/>
+        </geometry>
+      </collision>
+      <visual>
+        <origin xyz="0 0 0" rpy="0 0 0"/>
+        <geometry>
+          <mesh filename="package://ur_description/meshes/hokuyo.dae"/>
+        </geometry>
+      </visual>
+      <inertial>
+        <mass value="1e-5" />
+        <origin xyz="0 0 0" rpy="0 0 0"/>
+        <inertia ixx="1e-6" ixy="0" ixz="0" iyy="1e-6" iyz="0" izz="1e-6" />
+      </inertial>
+    </link>
+    <!-- laser joint -->
     <joint name="hokuyo_joint" type="fixed">
       <axis xyz="0 1 0" />
       <origin xyz="0 0 ${1 - 0.05/2}" rpy="0 0 0"/>
-      <parent link="${prefix}left_back_wheel"/>
+      <parent link="${prefix}base_link"/>
       <child link="hokuyo_link"/>
     </joint>
-    <!-- Hokuyo Laser -->
-    <link name="hokuyo_link">
-      <collision>
-        <origin xyz="0 0 0" rpy="0 0 0"/>
-        <geometry>
-          <box size="0.1 0.1 0.1"/>
-        </geometry>
-      </collision>
-      <visual>
-        <origin xyz="0 0 0" rpy="0 0 0"/>
-        <geometry>
-          <mesh filename="package://ur_description/meshes/hokuyo.dae"/>
-        </geometry>
-      </visual>
-      <inertial>
-        <mass value="1e-5" />
-        <origin xyz="0 0 0" rpy="0 0 0"/>
-        <inertia ixx="1e-6" ixy="0" ixz="0" iyy="1e-6" iyz="0" izz="1e-6" />
-      </inertial>
-    </link>
     <link name="${prefix}ur3_mount">
       <visual>

Commit message: lidar finished

File: Suii/suii_description/urdf/suii.xacro (robot description, xacro)
@@ -543,5 +543,5 @@
     </joint>
     <!-- Hokuyo Laser -->
-    <link name="hokuyo_link">
+    <link name="hokuyo_link_back">
       <collision>
         <origin xyz="0 0 0" rpy="0 0 0"/>
@@ -564,9 +564,37 @@
     </link>
     <!-- laser joint -->
-    <joint name="hokuyo_joint" type="fixed">
+    <joint name="hokuyo_joint_back" type="fixed">
       <axis xyz="0 1 0" />
-      <origin xyz="0.035 0 0.25" rpy="0 0 0"/>
+      <origin xyz="0.244 0.168 0.15" rpy="0 0 ${pi/4}"/>
       <parent link="${prefix}base_link"/>
-      <child link="hokuyo_link"/>
+      <child link="hokuyo_link_back"/>
+    </joint>
+    <!-- Hokuyo Laser -->
+    <link name="hokuyo_link_front">
+      <collision>
+        <origin xyz="0 0 0" rpy="0 0 0"/>
+        <geometry>
+          <box size="0.1 0.1 0.1"/>
+        </geometry>
+      </collision>
+      <visual>
+        <origin xyz="0 0 0" rpy="0 0 0"/>
+        <geometry>
+          <box size="${laser_link} ${laser_link} ${laser_link}"/>
+        </geometry>
+        <material name="red"/>
+      </visual>
+      <inertial>
+        <mass value="1e-5" />
+        <origin xyz="0 0 0" rpy="0 0 0"/>
+        <inertia ixx="1e-6" ixy="0" ixz="0" iyy="1e-6" iyz="0" izz="1e-6" />
+      </inertial>
+    </link>
+    <!-- laser joint -->
+    <joint name="hokuyo_joint_front" type="fixed">
+      <axis xyz="0 1 0" />
+      <origin xyz="-0.251153588295 -0.17189989984 0.16" rpy="0 0 ${pi/4 + pi}"/>
+      <parent link="${prefix}base_link"/>
+      <child link="hokuyo_link_front"/>
     </joint>
     <xacro:suii_transmission prefix="${prefix}" hw_interface="${transmission_hw_interface}" />

File: Suii/suii_description/urdf/suii_gazebo.xacro (robot description, xacro)
@@ -94,22 +94,22 @@
     </gazebo>
     <!-- hokuyo -->
-    <gazebo reference="hokuyo_link">
-      <sensor type="gpu_ray" name="head_hokuyo_sensor">
-        <pose>0 0 0 0 0 0</pose>
-        <visualize>false</visualize>
+    <gazebo reference="hokuyo_link_back">
+      <sensor type="gpu_ray" name="head_hokuyo_sensor_back">
+        <pose>0.244 0.168 0.15 0 0 0</pose>
+        <visualize>true</visualize>
         <update_rate>40</update_rate>
         <ray>
           <scan>
             <horizontal>
-              <samples>720</samples>
-              <resolution>1</resolution>
-              <min_angle>-1.570796</min_angle>
-              <max_angle>1.570796</max_angle>
+              <samples>1080</samples>
+              <resolution>0.25</resolution>
+              <min_angle>-2.35619449</min_angle>
+              <max_angle>2.35619449</max_angle>
             </horizontal>
           </scan>
           <range>
-            <min>0.10</min>
+            <min>0.06</min>
             <max>30.0</max>
-            <resolution>0.01</resolution>
+            <resolution>0.04</resolution>
           </range>
           <noise>
@@ -119,7 +119,39 @@
           </noise>
         </ray>
-        <plugin name="gazebo_ros_head_hokuyo_controller" filename="libgazebo_ros_gpu_laser.so">
-          <topicName>/suii/laser/scan</topicName>
-          <frameName>hokuyo_link</frameName>
+        <plugin name="gazebo_ros_head_hokuyo_controller_back" filename="libgazebo_ros_gpu_laser.so">
+          <topicName>/suii/laser/scan_back</topicName>
+          <frameName>hokuyo_link_back</frameName>
+        </plugin>
+      </sensor>
+    </gazebo>
+    <!-- hokuyo -->
+    <gazebo reference="hokuyo_link_front">
+      <sensor type="gpu_ray" name="head_hokuyo_sensor_front">
+        <pose>-0.244 -0.158 0.15 0 0 0</pose>
+        <visualize>true</visualize>
+        <update_rate>40</update_rate>
+        <ray>
+          <scan>
+            <horizontal>
+              <samples>1080</samples>
+              <resolution>0.25</resolution>
+              <min_angle>-2.35619449</min_angle>
+              <max_angle>2.35619449</max_angle>
+            </horizontal>
+          </scan>
+          <range>
+            <min>0.06</min>
+            <max>30.0</max>
+            <resolution>0.04</resolution>
+          </range>
+          <noise>
+            <type>gaussian</type>
+            <mean>0.0</mean>
+            <stddev>0.01</stddev>
+          </noise>
+        </ray>
+        <plugin name="gazebo_ros_head_hokuyo_controller_front" filename="libgazebo_ros_gpu_laser.so">
+          <topicName>/suii/laser/scan_front</topicName>
+          <frameName>hokuyo_link_front</frameName>
         </plugin>
       </sensor>
