Commit message: gripper base added

File: Suii/suii_description/urdf/suii.xacro (robot description, xacro)
@@ -476,13 +476,34 @@
       </xacro:cylinder_inertial>
     </link>
-    <!-- <joint name="${prefix}ee_fixed_joint" type="fixed">
+    <joint name="${prefix}gripper_mount" type="continuous">
       <parent link="${prefix}wrist_3_link" />
-      <child link = "${prefix}ee_link" />
-      <origin xyz="0.0 ${wrist_3_length} 0.0" rpy="0.0 0.0 ${pi/2.0}" />
-    </joint> -->
-    <joint name="${prefix}gripper_mount" type="revolute">
-      <parent link="${prefix}wrist_3_link" />
-      <child link = "${prefix}base_gripper" />
-      <origin xyz="0.0 0.085 ${wrist_3_length}" rpy="1.57 1.57 0" />
+      <child link = "${prefix}gripper_base" />
+      <origin xyz="0 0.08 ${wrist_3_length}" rpy="0 -1.57 0" />
+      <axis xyz="0 1 0" />
+    </joint>
+    <link name="${prefix}gripper_base">
+      <visual>
+        <geometry>
+          <mesh filename="package://suii_description/meshes/suii/visual/gripper_base.stl"/>
+        </geometry>
+        <material name="LightGrey">
+          <color rgba="0.7 0.7 0.7 1.0"/>
+        </material>
+      </visual>
+      <collision>
+        <geometry>
+          <mesh filename="package://suii_description/meshes/suii/collision/gripper_base.stl"/>
+        </geometry>
+      </collision>
+      <inertial>
+        <mass value= "${frame_mass}"/>
+        <inertia ixx="0.0" ixy="0.0" ixz="0.0" iyy="0" iyz="0" izz="0"/>
+        <origin xyz="0 0 0"  rpy="0 0 0" />
+      </inertial>
+    </link>
+    <!-- <joint name="${prefix}rightTilted_link" type="revolute">
+      <parent link="${prefix}gripper_base" />
+      <child link = "${prefix}rightTilted_link" />
+      <origin xyz="-0.04625 0.0035 -0.041" rpy="0 0 3.1416" />
       <axis xyz="0 1 0" />
       <xacro:unless value="${joint_limited}">
@@ -500,16 +521,16 @@
       <dynamics damping="0.0" friction="0.0"/>
     </joint>
-    <link name="${prefix}base_gripper">
-      <visual>
-        <geometry>
-          <mesh filename="package://suii_description/meshes/suii/visual/base_gripper.stl"/>
-        </geometry>
-        <material name="LightGrey">
-          <color rgba="0.7 0.7 0.7 1.0"/>
-        </material>
-      </visual>
-      <collision>
-        <geometry>
-          <mesh filename="package://suii_description/meshes/suii/collision/base_gripper.stl"/>
+    <link name="${prefix}rightTilted_link">
+      <visual>
+        <geometry>
+          <mesh filename="package://suii_description/meshes/suii/visual/rightTilted_link.stl"/>
+        </geometry>
+        <material name="LightGrey">
+          <color rgba="0.7 0.7 0.7 1.0"/>
+        </material>
+      </visual>
+      <collision>
+        <geometry>
+          <mesh filename="package://suii_description/meshes/suii/collision/rightTilted_link.stl"/>
         </geometry>
       </collision>
@@ -520,11 +541,111 @@
       </inertial>
     </link>
-<!--  -->
-    <joint name="${prefix}servo_link" type="fixed">
+    <joint name="${prefix}rightStraight_link" type="continuous">
+      <parent link="${prefix}gripper_base" />
+      <child link = "${prefix}rightStraight_link" />
+      <origin xyz="-0.02125 0.0035 -0.061" rpy="0 0 3.1416" />
+      <axis xyz="0 1 0" />  -->
+      <!-- <xacro:unless value="${joint_limited}">
+        <limit lower="${-2.0 * pi}" upper="${2.0 * pi}" effort="54.0" velocity="3.2"/>
+        <xacro:if value="${safety_limits}">
+          <safety_controller soft_lower_limit="${-2.0 * pi + safety_pos_margin}" soft_upper_limit="${2.0 * pi - safety_pos_margin}" k_position="${safety_k_position}" k_velocity="0.0"/>
+        </xacro:if>
+      </xacro:unless>
+      <xacro:if value="${joint_limited}">
+        <limit lower="${wrist_3_lower_limit}" upper="${wrist_3_upper_limit}" effort="54.0" velocity="3.2"/>
+        <xacro:if value="${safety_limits}">
+          <safety_controller soft_lower_limit="${wrist_3_lower_limit + safety_pos_margin}" soft_upper_limit="${wrist_3_upper_limit - safety_pos_margin}" k_position="${safety_k_position}" k_velocity="0.0"/>
+        </xacro:if>
+      </xacro:if>
+      <dynamics damping="0.0" friction="0.0"/>  -->
+    <!-- </joint>
+    <link name="${prefix}rightStraight_link">
+      <visual>
+        <geometry>
+          <mesh filename="package://suii_description/meshes/suii/visual/rightStraight_link.stl"/>
+        </geometry>
+        <material name="LightGrey">
+          <color rgba="0.7 0.7 0.7 1.0"/>
+        </material>
+      </visual>
+      <collision>
+        <geometry>
+          <mesh filename="package://suii_description/meshes/suii/collision/rightStraight_link.stl"/>
+        </geometry>
+      </collision>
+      <inertial>
+        <mass value= "${frame_mass}"/>
+        <inertia ixx="0.0" ixy="0.0" ixz="0.0" iyy="0" iyz="0" izz="0"/>
+        <origin xyz="0 0 0"  rpy="0 0 0" />
+      </inertial>
+    </link> -->
+ <!-- <joint name="${prefix}fingerRightLeft_link" type="continuous">
+       <parent link="${prefix}rightStraight_link" />
+      <child link = "${prefix}fingerRightLeft_link" />
+      <origin xyz="0.0838 0 -0.0102" rpy="0 0.2617 0"/>
+       <axis xyz="0 1 0" />
+      <parent link="${prefix}rightTilted_link" />
+      <child link = "${prefix}fingerRightLeft_link" />
+      <origin xyz="0.0579 0 -0.0302" />
+      <axis xyz="0 1 0" /> -->
+      <!-- <xacro:unless value="${joint_limited}">
+        <limit lower="${-2.0 * pi}" upper="${2.0 * pi}" effort="54.0" velocity="3.2"/>
+        <xacro:if value="${safety_limits}">
+          <safety_controller soft_lower_limit="${-2.0 * pi + safety_pos_margin}" soft_upper_limit="${2.0 * pi - safety_pos_margin}" k_position="${safety_k_position}" k_velocity="0.0"/>
+        </xacro:if>
+      </xacro:unless>
+      <xacro:if value="${joint_limited}">
+        <limit lower="${wrist_3_lower_limit}" upper="${wrist_3_upper_limit}" effort="54.0" velocity="3.2"/>
+        <xacro:if value="${safety_limits}">
+          <safety_controller soft_lower_limit="${wrist_3_lower_limit + safety_pos_margin}" soft_upper_limit="${wrist_3_upper_limit - safety_pos_margin}" k_position="${safety_k_position}" k_velocity="0.0"/>
+        </xacro:if>
+      </xacro:if>
+      <dynamics damping="0.0" friction="0.0"/>  -->
+    <!-- </joint>  -->
+ <!-- <joint name="${prefix}fingerRightLeft_link_2" type="continuous"> -->
+      <!-- <parent link="${prefix}rightStraight_link" />
+      <child link = "${prefix}fingerRightLeft_link" />
+      <origin xyz="0.0625 0 -0.0188" />
+      <axis xyz="0 1 0" /> -->
+      <!-- <xacro:unless value="${joint_limited}">
+        <limit lower="${-2.0 * pi}" upper="${2.0 * pi}" effort="54.0" velocity="3.2"/>
+        <xacro:if value="${safety_limits}">
+          <safety_controller soft_lower_limit="${-2.0 * pi + safety_pos_margin}" soft_upper_limit="${2.0 * pi - safety_pos_margin}" k_position="${safety_k_position}" k_velocity="0.0"/>
+        </xacro:if>
+      </xacro:unless>
+      <xacro:if value="${joint_limited}">
+        <limit lower="${wrist_3_lower_limit}" upper="${wrist_3_upper_limit}" effort="54.0" velocity="3.2"/>
+        <xacro:if value="${safety_limits}">
+          <safety_controller soft_lower_limit="${wrist_3_lower_limit + safety_pos_margin}" soft_upper_limit="${wrist_3_upper_limit - safety_pos_margin}" k_position="${safety_k_position}" k_velocity="0.0"/>
+        </xacro:if>
+      </xacro:if>
+      <dynamics damping="0.0" friction="0.0"/>  -->
+    <!-- </joint>  -->
+    <!-- <link name="${prefix}fingerRightLeft_link">
+      <visual>
+        <geometry>
+          <mesh filename="package://suii_description/meshes/suii/visual/fingerRightLeft_link.stl"/>
+        </geometry>
+        <material name="LightGrey">
+          <color rgba="0.7 0.7 0.7 1.0"/>
+        </material>
+      </visual>
+      <collision>
+        <geometry>
+          <mesh filename="package://suii_description/meshes/suii/collision/fingerRightLeft_link.stl"/>
+        </geometry>
+      </collision>
+      <inertial>
+        <mass value= "${frame_mass}"/>
+        <inertia ixx="0.0" ixy="0.0" ixz="0.0" iyy="0" iyz="0" izz="0"/>
+        <origin xyz="0 0 0"  rpy="0 0 0" />
+      </inertial>
+    </link> -->
+ <!-- <joint name="${prefix}leftStraight_link" type="revolute">
       <parent link="${prefix}base_gripper" />
-      <child link = "${prefix}servo_link" />
-      <origin xyz="0.0 0.1 0.0" rpy="1.57 1.57 0" />
-      <axis xyz="0 1 0" />
-      <!-- <xacro:unless value="${joint_limited}">
+      <child link = "${prefix}leftStraight_link" />
+      <origin xyz="0 0 0" rpy="0 0 0" />
+      <axis xyz="0 1 0" />
+      <xacro:unless value="${joint_limited}">
         <limit lower="${-2.0 * pi}" upper="${2.0 * pi}" effort="54.0" velocity="3.2"/>
         <xacro:if value="${safety_limits}">
@@ -538,18 +659,18 @@
         </xacro:if>
       </xacro:if>
-      <dynamics damping="0.0" friction="0.0"/> -->
-    </joint>
-    <link name="${prefix}servo_link">
-      <visual>
-        <geometry>
-          <mesh filename="package://suii_description/meshes/suii/visual/servo_link.stl"/>
-        </geometry>
-        <material name="LightGrey">
-          <color rgba="0.7 0.7 0.7 1.0"/>
-        </material>
-      </visual>
-      <collision>
-        <geometry>
-          <mesh filename="package://suii_description/meshes/suii/collision/servo_link.stl"/>
+      <dynamics damping="0.0" friction="0.0"/>
+    </joint>
+    <link name="${prefix}leftStraight_link">
+      <visual>
+        <geometry>
+          <mesh filename="package://suii_description/meshes/suii/visual/leftStraight_link.stl"/>
+        </geometry>
+        <material name="LightGrey">
+          <color rgba="0.7 0.7 0.7 1.0"/>
+        </material>
+      </visual>
+      <collision>
+        <geometry>
+          <mesh filename="package://suii_description/meshes/suii/collision/leftStraight_link.stl"/>
         </geometry>
       </collision>
@@ -560,4 +681,82 @@
       </inertial>
     </link>
+ <joint name="${prefix}leftTilted_link" type="revolute">
+      <parent link="${prefix}base_gripper" />
+      <child link = "${prefix}leftTilted_link" />
+      <origin xyz="0 0 0" rpy="0 0 0" />
+      <axis xyz="0 1 0" />
+      <xacro:unless value="${joint_limited}">
+        <limit lower="${-2.0 * pi}" upper="${2.0 * pi}" effort="54.0" velocity="3.2"/>
+        <xacro:if value="${safety_limits}">
+          <safety_controller soft_lower_limit="${-2.0 * pi + safety_pos_margin}" soft_upper_limit="${2.0 * pi - safety_pos_margin}" k_position="${safety_k_position}" k_velocity="0.0"/>
+        </xacro:if>
+      </xacro:unless>
+      <xacro:if value="${joint_limited}">
+        <limit lower="${wrist_3_lower_limit}" upper="${wrist_3_upper_limit}" effort="54.0" velocity="3.2"/>
+        <xacro:if value="${safety_limits}">
+          <safety_controller soft_lower_limit="${wrist_3_lower_limit + safety_pos_margin}" soft_upper_limit="${wrist_3_upper_limit - safety_pos_margin}" k_position="${safety_k_position}" k_velocity="0.0"/>
+        </xacro:if>
+      </xacro:if>
+      <dynamics damping="0.0" friction="0.0"/>
+    </joint>
+    <link name="${prefix}leftTilted_link">
+      <visual>
+        <geometry>
+          <mesh filename="package://suii_description/meshes/suii/visual/leftTilted_link.stl"/>
+        </geometry>
+        <material name="LightGrey">
+          <color rgba="0.7 0.7 0.7 1.0"/>
+        </material>
+      </visual>
+      <collision>
+        <geometry>
+          <mesh filename="package://suii_description/meshes/suii/collision/leftTilted_link.stl"/>
+        </geometry>
+      </collision>
+      <inertial>
+        <mass value= "${frame_mass}"/>
+        <inertia ixx="0.0" ixy="0.0" ixz="0.0" iyy="0" iyz="0" izz="0"/>
+        <origin xyz="0 0 0"  rpy="0 0 0" />
+      </inertial>
+    </link>
+ <joint name="${prefix}fingerLeftLeft_link" type="revolute">
+      <parent link="${prefix}base_gripper" />
+      <child link = "${prefix}fingerLeftLeft_link" />
+      <origin xyz="0 0 0" rpy="0 0 0" />
+      <axis xyz="0 1 0" />
+      <xacro:unless value="${joint_limited}">
+        <limit lower="${-2.0 * pi}" upper="${2.0 * pi}" effort="54.0" velocity="3.2"/>
+        <xacro:if value="${safety_limits}">
+          <safety_controller soft_lower_limit="${-2.0 * pi + safety_pos_margin}" soft_upper_limit="${2.0 * pi - safety_pos_margin}" k_position="${safety_k_position}" k_velocity="0.0"/>
+        </xacro:if>
+      </xacro:unless>
+      <xacro:if value="${joint_limited}">
+        <limit lower="${wrist_3_lower_limit}" upper="${wrist_3_upper_limit}" effort="54.0" velocity="3.2"/>
+        <xacro:if value="${safety_limits}">
+          <safety_controller soft_lower_limit="${wrist_3_lower_limit + safety_pos_margin}" soft_upper_limit="${wrist_3_upper_limit - safety_pos_margin}" k_position="${safety_k_position}" k_velocity="0.0"/>
+        </xacro:if>
+      </xacro:if>
+      <dynamics damping="0.0" friction="0.0"/>
+    </joint>
+    <link name="${prefix}fingerLeftLeft_link">
+      <visual>
+        <geometry>
+          <mesh filename="package://suii_description/meshes/suii/visual/fingerLeftLeft_link.stl"/>
+        </geometry>
+        <material name="LightGrey">
+          <color rgba="0.7 0.7 0.7 1.0"/>
+        </material>
+      </visual>
+      <collision>
+        <geometry>
+          <mesh filename="package://suii_description/meshes/suii/collision/fingerLeftLeft_link.stl"/>
+        </geometry>
+      </collision>
+      <inertial>
+        <mass value= "${frame_mass}"/>
+        <inertia ixx="0.0" ixy="0.0" ixz="0.0" iyy="0" iyz="0" izz="0"/>
+        <origin xyz="0 0 0"  rpy="0 0 0" />
+      </inertial>
+    </link> -->
     <!-- <link name="${prefix}ee_link">
       <collision>

File: Suii_Gripper/urdf/gripper.urdf (robot description, URDF)
Before this commit: robot gripper, 7 links, 7 joints
Links:
- added link base_link, mass 1.15466628725613; collision mesh filename=package://suii_gripper/meshes/base_link.STL; visual mesh filename=package://suii_gripper/meshes/base_link.STL
