Commit message: everything added, except ur_modern_driver and universal_robot

File: Suii/suii_description/urdf/suii.xacro (robot description, xacro)
@@ -57,4 +57,9 @@
     <xacro:property name="wrist_2_length" value="${d5}" />
     <xacro:property name="wrist_3_length" value="${d6}" />
+    <!-- sensor properties-->
+    <xacro:property name="sonar_link" value="-0.05" /> <!-- Size of square 'sonar' box -->
+    <xacro:property name="laser_link" value="-0.05" /> <!-- Size of square 'sonar' box -->
+    <xacro:property name="height" value="0.3" /> <!-- height sensors-->
+    <xacro:property name="axel_offset" value="0.05" /> <!-- offset placement -->
     <gazebo>
 	    <plugin name="omni_steering" filename="libgazebo_ros_planar_move.so">
@@ -496,17 +501,315 @@
       </xacro:cylinder_inertial>
     </link>
-    <joint name="${prefix}ee_fixed_joint" type="fixed">
+    <joint name="${prefix}wrist_3_link" type="revolute">
       <parent link="${prefix}wrist_3_link" />
-      <child link = "${prefix}ee_link" />
-      <origin xyz="0.0 ${wrist_3_length} 0.0" rpy="0.0 0.0 ${pi/2.0}" />
-    </joint>
-    <link name="${prefix}ee_link">
-      <collision>
-        <geometry>
-          <box size="0.01 0.01 0.01"/>
-        </geometry>
-        <origin rpy="0 0 0" xyz="-0.01 0 0"/>
-      </collision>
-    </link>
+      <child link = "${prefix}gripper_base" />1.4771E-10
+      <origin xyz="0 0.085 0" rpy="0 1.57 -1.57" />
+      <axis xyz="0 1 0" />
+      <xacro:unless value="${joint_limited}">
+        <limit lower="${-2.0 * pi}" upper="${2.0 * pi}" effort="54.0" velocity="3.2"/>
+        <xacro:if value="${safety_limits}">
+          <safety_controller soft_lower_limit="${-2.0 * pi + safety_pos_margin}" soft_upper_limit="${2.0 * pi - safety_pos_margin}" k_position="${safety_k_position}" k_velocity="0.0"/>
+        </xacro:if>
+      </xacro:unless>
+      <xacro:if value="${joint_limited}">
+        <limit lower="${wrist_3_lower_limit}" upper="${wrist_3_upper_limit}" effort="54.0" velocity="3.2"/>
+        <xacro:if value="${safety_limits}">
+          <safety_controller soft_lower_limit="${wrist_3_lower_limit + safety_pos_margin}" soft_upper_limit="${wrist_3_upper_limit - safety_pos_margin}" k_position="${safety_k_position}" k_velocity="0.0"/>
+        </xacro:if>
+      </xacro:if>
+      <dynamics damping="0.0" friction="0.0"/>
+    </joint>
+    <link name="${prefix}gripper_base">
+      <visual>
+        <geometry>
+          <mesh filename="package://suii_description/meshes/suii/visual/gripper_base.STL"/>
+        </geometry>
+        <material name="LightGrey">
+          <color rgba="0.7 0.7 0.7 1.0"/>
+        </material>
+      </visual>
+      <collision>
+        <geometry>
+          <mesh filename="package://suii_description/meshes/suii/collision/gripper_base.STL"/>
+        </geometry>
+      </collision>
+      <inertial>
+        <mass value= "${frame_mass}"/>
+        <inertia ixx="0.0" ixy="0.0" ixz="0.0" iyy="0" iyz="0" izz="0"/>
+        <origin xyz="0 0 0"  rpy="0 0 0" />
+      </inertial>
+    </link>
+    <link name="${prefix}leftTilted_link">
+      <visual>
+        <geometry>
+          <mesh filename="package://suii_description/meshes/suii/visual/leftTilted_link.STL"/>
+        </geometry>
+        <material name="LightGrey">
+          <color rgba="0.7 0.7 0.7 1.0"/>
+        </material>
+      </visual>
+      <collision>
+        <geometry>
+          <mesh filename="package://suii_description/meshes/suii/collision/leftTilted_link.STL"/>
+        </geometry>
+      </collision>
+      <inertial>
+        <mass value= "${frame_mass}"/>
+        <inertia ixx="0.0" ixy="0.0" ixz="0.0" iyy="0" iyz="0" izz="0"/>
+        <origin xyz="0 0 0"  rpy="0 0 0" />
+      </inertial>
+    </link>
+    <joint name="${prefix}leftTilted_link" type="revolute">
+      <parent link="${prefix}gripper_base" />
+      <child link = "${prefix}leftTilted_link" />
+      <origin xyz="0.04625 0.0035 -0.041" rpy="${pi} ${pi} 0" />
+      <axis xyz="0 1 0" />
+      <limit lower="${-1.6}" upper="${0}" effort="54.0" velocity="3.2"/>
+      <dynamics damping="0.0" friction="0.0"/>
+    </joint>
+     <link name="${prefix}rightTilted_link">
+      <visual>
+        <geometry>
+          <mesh filename="package://suii_description/meshes/suii/visual/rightTilted_link.STL"/>
+        </geometry>
+        <material name="LightGrey">
+          <color rgba="0.7 0.7 0.7 1.0"/>
+        </material>
+      </visual>
+      <collision>
+        <geometry>
+          <mesh filename="package://suii_description/meshes/suii/collision/rightTilted_link.STL"/>
+        </geometry>
+      </collision>
+      <inertial>
+        <mass value= "${frame_mass}"/>
+        <inertia ixx="0.0" ixy="0.0" ixz="0.0" iyy="0" iyz="0" izz="0"/>
+        <origin xyz="0 0 0"  rpy="0 0 0" />
+      </inertial>
+    </link>
+    <joint name="${prefix}rightTilted_link" type="revolute">
+      <parent link="${prefix}gripper_base" />
+      <child link = "${prefix}rightTilted_link" />
+      <origin xyz="-0.04625 0.0035 -0.041" rpy="${pi} ${pi} 0" />
+      <axis xyz="0 1 0" />
+      <limit lower="${0}" upper="${1.6}" effort="54.0" velocity="3.2"/>
+      <dynamics damping="0.0" friction="0.0"/>
+    </joint>
+    <link name="${prefix}rightStraight_link">
+      <visual>
+        <geometry>
+          <mesh filename="package://suii_description/meshes/suii/visual/rightStraight_link.STL"/>
+        </geometry>
+        <material name="LightGrey">
+          <color rgba="0.7 0.7 0.7 1.0"/>
+        </material>
+      </visual>
+      <collision>
+        <geometry>
+          <mesh filename="package://suii_description/meshes/suii/collision/rightStraight_link.STL"/>
+        </geometry>
+      </collision>
+      <inertial>
+        <mass value= "${frame_mass}"/>
+        <inertia ixx="0.0" ixy="0.0" ixz="0.0" iyy="0" iyz="0" izz="0"/>
+        <origin xyz="0 0 0"  rpy="0 0 0" />
+      </inertial>
+    </link>
+    <joint name="${prefix}rightStraight_link" type="revolute">
+      <parent link="${prefix}gripper_base" />
+      <child link = "${prefix}rightStraight_link" />
+      <origin xyz="-0.02125 0.0035 -0.061" rpy="${pi} ${pi} 0" />
+      <axis xyz="0 1 0" />
+      <limit lower="${0}" upper="${1.6}" effort="54.0" velocity="3.2"/>
+      <dynamics damping="0.0" friction="0.0"/>
+    </joint>
+    <link name="${prefix}leftStraight_link">
+      <visual>
+        <geometry>
+          <mesh filename="package://suii_description/meshes/suii/visual/leftStraight_link.STL"/>
+        </geometry>
+        <material name="LightGrey">
+          <color rgba="0.7 0.7 0.7 1.0"/>
+        </material>
+      </visual>
+      <collision>
+        <geometry>
+          <mesh filename="package://suii_description/meshes/suii/collision/leftStraight_link.STL"/>
+        </geometry>
+      </collision>
+      <inertial>
+        <mass value= "${frame_mass}"/>
+        <inertia ixx="0.0" ixy="0.0" ixz="0.0" iyy="0" iyz="0" izz="0"/>
+        <origin xyz="0 0 0"  rpy="0 0 0" />
+      </inertial>
+    </link>
+    <joint name="${prefix}leftStraight_link" type="revolute">
+      <parent link="${prefix}gripper_base" />
+      <child link = "${prefix}leftStraight_link" />
+      <origin xyz="0.02125 0.0035 -0.061" rpy="${pi} ${pi} 0" />
+      <axis xyz="0 1 0" />
+      <limit lower="${-1.6}" upper="${0}" effort="54.0" velocity="3.2"/>
+      <dynamics damping="0.0" friction="0.0"/>
+    </joint>
+    <link name="${prefix}right_finger">
+      <visual>
+        <geometry>
+          <mesh filename="package://suii_description/meshes/suii/visual/finger.STL"/>
+        </geometry>
+        <material name="LightGrey">
+          <color rgba="0.7 0.7 0.7 1.0"/>
+        </material>
+      </visual>
+      <collision>
+        <geometry>
+          <mesh filename="package://suii_description/meshes/suii/collision/finger.STL"/>
+        </geometry>
+      </collision>
+      <inertial>
+        <mass value= "${frame_mass}"/>
+        <inertia ixx="0.0" ixy="0.0" ixz="0.0" iyy="0" iyz="0" izz="0"/>
+        <origin xyz="0 0 0"  rpy="0 0 0" />
+      </inertial>
+    </link>
+    <joint name="${prefix}right_finger" type="revolute">
+      <parent link="${prefix}rightTilted_link" />
+      <child link = "${prefix}right_finger" />
+      <origin xyz="0.07358 0.01 -0.01452" rpy="${pi} ${pi} 0" />
+      <axis xyz="0 1 0" />
+      <limit lower="${0}" upper="${1.6}" effort="54.0" velocity="3.2"/>
+      <dynamics damping="0.0" friction="0.0"/>
+    </joint>
+    <link name="${prefix}left_finger">
+      <visual>
+        <geometry>
+          <mesh filename="package://suii_description/meshes/suii/visual/finger.STL"/>
+        </geometry>
+        <material name="LightGrey">
+          <color rgba="0.7 0.7 0.7 1.0"/>
+        </material>
+      </visual>
+      <collision>
+        <geometry>
+          <mesh filename="package://suii_description/meshes/suii/collision/finger.STL"/>
+        </geometry>
+      </collision>
+      <inertial>
+        <mass value= "${frame_mass}"/>
+        <inertia ixx="0.0" ixy="0.0" ixz="0.0" iyy="0" iyz="0" izz="0"/>
+        <origin xyz="0 0 0"  rpy="0 0 0" />
+      </inertial>
+    </link>
+    <joint name="${prefix}left_finger" type="revolute">
+      <parent link="${prefix}leftTilted_link" />
+      <child link = "${prefix}left_finger" />
+      <origin xyz="-0.07358 -0.01 -0.01452" rpy="${pi} ${pi} ${pi}" />
+      <axis xyz="0 1 0" />
+      <limit lower="${0}" upper="${1.6}" effort="54.0" velocity="3.2"/>
+      <dynamics damping="0.0" friction="0.0"/>
+    </joint>
+    <gazebo>
+ 	 <plugin name="mimic" filename="libroboticsgroup_gazebo_mimic_joint_plugin.so">
+	    <joint>${prefix}leftTilted_link</joint>
+	    <mimicJoint>${prefix}leftStraight_link</mimicJoint>
+            <multiplier>1</multiplier>
+	 </plugin>
+    </gazebo>
+    <gazebo>
+ 	 <plugin name="mimic2" filename="libroboticsgroup_gazebo_mimic_joint_plugin.so">
+	    <joint>${prefix}rightTilted_link</joint>
+	    <mimicJoint>${prefix}rightStraight_link</mimicJoint>
+            <multiplier>1</multiplier>
+	 </plugin>
+    </gazebo>
+    <gazebo>
+ 	 <plugin name="mimic3" filename="libroboticsgroup_gazebo_mimic_joint_plugin.so">
+	    <joint>${prefix}leftTilted_link</joint>
+	    <mimicJoint>${prefix}left_finger</mimicJoint>
+            <multiplier>-1</multiplier>
+	 </plugin>
+    </gazebo>
+    <gazebo>
+ 	 <plugin name="mimic4" filename="libroboticsgroup_gazebo_mimic_joint_plugin.so">
+	    <joint>${prefix}rightTilted_link</joint>
+	    <mimicJoint>${prefix}right_finger</mimicJoint>
+            <multiplier>1</multiplier>
+	 </plugin>
+    </gazebo>
+    <link name="sonar_link">
+      <collision>
+        <origin xyz="0 0 0" rpy="0 0 0"/>
+        <geometry>
+          <mesh filename="package://suii_description/meshes/suii/collision/leftStraight_link.stl"/>
+        </geometry>
+      </collision>
+      <inertial>
+        <mass value= "${frame_mass}"/>
+        <inertia ixx="0.0" ixy="0.0" ixz="0.0" iyy="0" iyz="0" izz="0"/>
+        <origin xyz="0 0 0"  rpy="0 0 0" />
+      </inertial>
+    </link>
+    <!-- sonar joint -->
+    <joint name="sonar_joint" type="fixed">
+      <axis xyz= "0 1 0" />
+      <origin xyz="-0.275 0 0.1" rpy="0 0 3.1415926535897931"/>
+      <parent link="${prefix}base_link"/>
+      <child link="sonar_link"/>
+    </joint>
+    <!-- Hokuyo Laser -->
+    <link name="hokuyo_link_back">
+      <collision>
+        <origin xyz="0 0 0" rpy="0 0 0"/>
+        <geometry>
+          <box size="0.1 0.1 0.1"/>
+        </geometry>
+      </collision>
+      <visual>
+        <origin xyz="0 0 0" rpy="0 0 0"/>
+        <geometry>
+          <box size="${laser_link} ${laser_link} ${laser_link}"/>
+        </geometry>
+        <material name="red"/>
+      </visual>
+      <inertial>
+        <mass value="1e-5" />
+        <origin xyz="0 0 0" rpy="0 0 0"/>
+        <inertia ixx="1e-6" ixy="0" ixz="0" iyy="1e-6" iyz="0" izz="1e-6" />
+      </inertial>
+    </link>
+    <!-- laser joint -->
+    <joint name="hokuyo_joint_back" type="fixed">
+      <axis xyz="0 1 0" />
+      <origin xyz="0.244 0.168 0.15" rpy="0 0 ${pi/4}"/>
+      <parent link="${prefix}base_link"/>
+      <child link="hokuyo_link_back"/>
+    </joint>
+    <!-- Hokuyo Laser -->
+    <link name="hokuyo_link_front">
+      <collision>
+        <origin xyz="0 0 0" rpy="0 0 0"/>
+        <geometry>
+          <box size="0.1 0.1 0.1"/>
+        </geometry>
+      </collision>
+      <visual>
+        <origin xyz="0 0 0" rpy="0 0 0"/>
+        <geometry>
+          <box size="${laser_link} ${laser_link} ${laser_link}"/>
+        </geometry>
+        <material name="red"/>
+      </visual>
+      <inertial>
+        <mass value="1e-5" />
+        <origin xyz="0 0 0" rpy="0 0 0"/>
+        <inertia ixx="1e-6" ixy="0" ixz="0" iyy="1e-6" iyz="0" izz="1e-6" />
+      </inertial>
+    </link>
+    <!-- laser joint -->
+    <joint name="hokuyo_joint_front" type="fixed">
+      <axis xyz="0 1 0" />
+      <origin xyz="-0.251153588295 -0.17189989984 0.16" rpy="0 0 ${pi/4 + pi}"/>
+      <parent link="${prefix}base_link"/>
+      <child link="hokuyo_link_front"/>
+    </joint>
     <xacro:suii_transmission prefix="${prefix}" hw_interface="${transmission_hw_interface}" />
     <xacro:suii_gazebo prefix="${prefix}" />

File: Suii/suii_description/urdf/suii_transmission.xacro (robot description, xacro)
@@ -65,4 +65,67 @@
       </actuator>
     </transmission>
+    <transmission name="${prefix}wrist_3_trans">
+      <type>transmission_interface/SimpleTransmission</type>
+      <joint name="${prefix}wrist_3_joint">
+        <hardwareInterface>${hw_interface}</hardwareInterface>
+      </joint>
+      <actuator name="${prefix}wrist_3_motor">
+        <mechanicalReduction>1</mechanicalReduction>
+      </actuator>
+    </transmission>
+    <transmission name="${prefix}leftTilted_link_trans">
+      <type>transmission_interface/SimpleTransmission</type>
+      <joint name="${prefix}leftTilted_link">
+        <hardwareInterface>${hw_interface}</hardwareInterface>
+      </joint>
+      <actuator name="${prefix}leftTilted_link_motor">
+        <mechanicalReduction>1</mechanicalReduction>
+      </actuator>
+    </transmission>
+    <transmission name="${prefix}rightTilted_link_trans">
+      <type>transmission_interface/SimpleTransmission</type>
+      <joint name="${prefix}rightTilted_link">
+        <hardwareInterface>${hw_interface}</hardwareInterface>
+      </joint>
+      <actuator name="${prefix}rightTilted_link_motor">
+        <mechanicalReduction>1</mechanicalReduction>
+      </actuator>
+    </transmission>
+    <transmission name="${prefix}leftStraight_link_trans">
+      <type>transmission_interface/SimpleTransmission</type>
+      <joint name="${prefix}leftStraight_link">
+        <hardwareInterface>${hw_interface}</hardwareInterface>
+      </joint>
+      <actuator name="${prefix}leftStraight_link_motor">
+        <mechanicalReduction>1</mechanicalReduction>
+      </actuator>
+    </transmission>
+    <transmission name="${prefix}rightStraight_link_trans">
+      <type>transmission_interface/SimpleTransmission</type>
+      <joint name="${prefix}rightStraight_link">
+        <hardwareInterface>${hw_interface}</hardwareInterface>
+      </joint>
+      <actuator name="${prefix}rightStraight_link_motor">
+        <mechanicalReduction>1</mechanicalReduction>
+      </actuator>
+    </transmission>
+    <transmission name="${prefix}right_finger_trans">
+      <type>transmission_interface/SimpleTransmission</type>
+      <joint name="${prefix}right_finger">
+        <hardwareInterface>${hw_interface}</hardwareInterface>
+      </joint>
+      <actuator name="${prefix}right_finger_motor">
+        <mechanicalReduction>1</mechanicalReduction>
+      </actuator>
+    </transmission>
+    <transmission name="${prefix}left_finger_trans">
+      <type>transmission_interface/SimpleTransmission</type>
+      <joint name="${prefix}left_finger">
+        <hardwareInterface>${hw_interface}</hardwareInterface>
+      </joint>
+      <actuator name="${prefix}left_finger_motor">
+        <mechanicalReduction>1</mechanicalReduction>
+      </actuator>
+    </transmission>
   </xacro:macro>
 </robot>

Commit message: edit inertial

File: Suii/suii_description/urdf/suii.xacro (robot description, xacro)
@@ -32,5 +32,10 @@
     <xacro:property name="wrist_3_mass" value="0.35"/>
     <xacro:property name="frame_mass" value="20.5"/>
+    <xacro:property name="ur3_mount_plate" value="0.08"/>
     <xacro:property name="wheel_mass" value="0.37904"/>
+    <xacro:property name="gripper_base_mass" value="0.500"/>
+    <xacro:property name="Tilted_link" value="0.035"/>
+    <!-- <xacro:property name="" value="0.500"/>
+    <xacro:property name="" value="0.500"/> -->
     <xacro:property name="shoulder_cog" value="0.0 -0.02 0.0" />
     <xacro:property name="upper_arm_cog" value="0.13 0.0 0.1157" />
@@ -108,5 +113,5 @@
       <inertial>
         <mass value= "${frame_mass}"/>
-        <inertia ixx="0.0" ixy="0.0" ixz="0.0" iyy="0" iyz="0" izz="0"/>
+        <inertia ixx="0.34725" ixy="0.012191" ixz="1.1509E-06" iyy="0.91352" iyz="1.7554E-06" izz="0.66499"/>
         <origin xyz="0.15 -0.000252178578867549 0.0919059339213158"  rpy="0 0 0" />
       </inertial>
@@ -133,6 +138,6 @@
       </collision>
       <inertial>
-        <mass value= "${bottom_mass}"/>
-        <inertia ixx="0.0" ixy="0.0" ixz="0.0" iyy="0" iyz="0" izz="0"/>
+        <mass value= "${ur3_mount_plate}"/>
+        <inertia ixx="0.00013877" ixy="1.8488E-22" ixz="-3.1995E-06" iyy="0.00027709" iyz="-3.5837E-22" izz="-3.5837E-22"/>
         <origin xyz="0.0 0.0 0.0"  rpy="0 0 0" />
       </inertial>
@@ -160,5 +165,5 @@
       <inertial>
         <mass value= "${wheel_mass}"/>
-        <inertia ixx="0.0" ixy="0.0" ixz="0.0" iyy="0" iyz="0" izz="0"/>
+        <inertia ixx="0.00037409" ixy="2.9355E-20" ixz="2.4641E-12" iyy="0.00037409" iyz="4.7724E-12" izz="0.00061547"/>
         <origin xyz="6.3835E-11 -1.4771E-10 -0.030043"  rpy="0 0 0" />
       </inertial>
@@ -186,5 +191,5 @@
       <inertial>
         <mass value= "${wheel_mass}"/>
-        <inertia ixx="0.0" ixy="0.0" ixz="0.0" iyy="0" iyz="0" izz="0"/>
+        <inertia ixx="0.00037409" ixy="2.9355E-20" ixz="2.4641E-12" iyy="0.00037409" iyz="4.7724E-12" izz="0.00061547"/>
         <origin xyz="6.3835E-11 -1.4771E-10 -0.030043"  rpy="0 0 0" />
       </inertial>
@@ -212,5 +217,5 @@
       <inertial>
         <mass value= "${wheel_mass}"/>
-        <inertia ixx="0.0" ixy="0.0" ixz="0.0" iyy="0" iyz="0" izz="0"/>
+        <inertia ixx="0.00037409" ixy="2.9355E-20" ixz="2.4641E-12" iyy="0.00037409" iyz="4.7724E-12" izz="0.00061547"/>
         <origin xyz="6.3835E-11 -1.4771E-10 -0.030043"  rpy="0 0 0" />
       </inertial>
@@ -238,5 +243,5 @@
       <inertial>
         <mass value= "${wheel_mass}"/>
-        <inertia ixx="0.0" ixy="0.0" ixz="0.0" iyy="0" iyz="0" izz="0"/>
+        <inertia ixx="0.00037409" ixy="2.9355E-20" ixz="2.4641E-12" iyy="0.00037409" iyz="4.7724E-12" izz="0.00061547"/>
         <origin xyz="6.3835E-11 -1.4771E-10 -0.030043"  rpy="0 0 0" />
       </inertial>
@@ -535,6 +540,6 @@
       </collision>
       <inertial>
-        <mass value= "${frame_mass}"/>
-        <inertia ixx="0.0" ixy="0.0" ixz="0.0" iyy="0" iyz="0" izz="0"/>
+        <mass value= "${gripper_base_mass}"/>
+        <inertia ixx="3.1166E-10" ixy="-4.678E-12" ixz="1.861E-11" iyy="8.724E-10" iyz="5.6254E-11" izz="6.5089E-10"/>
         <origin xyz="0 0 0"  rpy="0 0 0" />
       </inertial>
