Commit message: merge with alfredo

File: Suii/suii_description/urdf/suii.xacro (robot description, xacro)
@@ -35,7 +35,7 @@
     <xacro:property name="wheel_mass" value="0.37904"/>
     <xacro:property name="gripper_base_mass" value="0.500"/>
-    <xacro:property name="Tilted_link_mass" value="0.035"/>
-    <xacro:property name="straight_link_mass" value="0.042"/>
-    <xacro:property name="finger_mass" value="0.035"/>
+    <xacro:property name="Tilted_link" value="0.035"/>
+    <!-- <xacro:property name="" value="0.500"/>
+    <xacro:property name="" value="0.500"/> -->
     <xacro:property name="shoulder_cog" value="0.0 -0.02 0.0" />
     <xacro:property name="upper_arm_cog" value="0.13 0.0 0.1157" />
@@ -550,16 +550,5 @@
       <origin xyz="0.04625 0.0035 -0.041" rpy="${pi} ${pi} 0" />
       <axis xyz="0 1 0" />
-      <xacro:unless value="${joint_limited}">
-        <limit lower="${-2.0 * pi}" upper="${2.0 * pi}" effort="54.0" velocity="3.2"/>
-        <xacro:if value="${safety_limits}">
-          <safety_controller soft_lower_limit="${-2.0 * pi + safety_pos_margin}" soft_upper_limit="${2.0 * pi - safety_pos_margin}" k_position="${safety_k_position}" k_velocity="0.0"/>
-        </xacro:if>
-      </xacro:unless>
-      <xacro:if value="${joint_limited}">
-        <limit lower="${wrist_3_lower_limit}" upper="${wrist_3_upper_limit}" effort="54.0" velocity="3.2"/>
-        <xacro:if value="${safety_limits}">
-          <safety_controller soft_lower_limit="${wrist_3_lower_limit + safety_pos_margin}" soft_upper_limit="${wrist_3_upper_limit - safety_pos_margin}" k_position="${safety_k_position}" k_velocity="0.0"/>
-        </xacro:if>
-      </xacro:if>
+      <limit lower="${-1.6}" upper="${0}" effort="54.0" velocity="3.2"/>
       <dynamics damping="0.0" friction="0.0"/>
     </joint>
@@ -589,16 +578,5 @@
       <origin xyz="-0.04625 0.0035 -0.041" rpy="${pi} ${pi} 0" />
       <axis xyz="0 1 0" />
-      <xacro:unless value="${joint_limited}">
-        <limit lower="${-2.0 * pi}" upper="${2.0 * pi}" effort="54.0" velocity="3.2"/>
-        <xacro:if value="${safety_limits}">
-          <safety_controller soft_lower_limit="${-2.0 * pi + safety_pos_margin}" soft_upper_limit="${2.0 * pi - safety_pos_margin}" k_position="${safety_k_position}" k_velocity="0.0"/>
-        </xacro:if>
-      </xacro:unless>
-      <xacro:if value="${joint_limited}">
-        <limit lower="${wrist_3_lower_limit}" upper="${wrist_3_upper_limit}" effort="54.0" velocity="3.2"/>
-        <xacro:if value="${safety_limits}">
-          <safety_controller soft_lower_limit="${wrist_3_lower_limit + safety_pos_margin}" soft_upper_limit="${wrist_3_upper_limit - safety_pos_margin}" k_position="${safety_k_position}" k_velocity="0.0"/>
-        </xacro:if>
-      </xacro:if>
+      <limit lower="${0}" upper="${1.6}" effort="54.0" velocity="3.2"/>
       <dynamics damping="0.0" friction="0.0"/>
     </joint>
@@ -628,16 +606,5 @@
       <origin xyz="-0.02125 0.0035 -0.061" rpy="${pi} ${pi} 0" />
       <axis xyz="0 1 0" />
-      <xacro:unless value="${joint_limited}">
-        <limit lower="${-2.0 * pi}" upper="${2.0 * pi}" effort="54.0" velocity="3.2"/>
-        <xacro:if value="${safety_limits}">
-          <safety_controller soft_lower_limit="${-2.0 * pi + safety_pos_margin}" soft_upper_limit="${2.0 * pi - safety_pos_margin}" k_position="${safety_k_position}" k_velocity="0.0"/>
-        </xacro:if>
-      </xacro:unless>
-      <xacro:if value="${joint_limited}">
-        <limit lower="${wrist_3_lower_limit}" upper="${wrist_3_upper_limit}" effort="54.0" velocity="3.2"/>
-        <xacro:if value="${safety_limits}">
-          <safety_controller soft_lower_limit="${wrist_3_lower_limit + safety_pos_margin}" soft_upper_limit="${wrist_3_upper_limit - safety_pos_margin}" k_position="${safety_k_position}" k_velocity="0.0"/>
-        </xacro:if>
-      </xacro:if>
+      <limit lower="${0}" upper="${1.6}" effort="54.0" velocity="3.2"/>
       <dynamics damping="0.0" friction="0.0"/>
     </joint>
@@ -662,21 +629,10 @@
       </inertial>
     </link>
-    <joint name="${prefix}lefStraight_link" type="revolute">
+    <joint name="${prefix}leftStraight_link" type="revolute">
       <parent link="${prefix}gripper_base" />
-      <child link = "${prefix}lefStraight_link" />
+      <child link = "${prefix}leftStraight_link" />
       <origin xyz="0.02125 0.0035 -0.061" rpy="${pi} ${pi} 0" />
       <axis xyz="0 1 0" />
-      <xacro:unless value="${joint_limited}">
-        <limit lower="${-2.0 * pi}" upper="${2.0 * pi}" effort="54.0" velocity="3.2"/>
-        <xacro:if value="${safety_limits}">
-          <safety_controller soft_lower_limit="${-2.0 * pi + safety_pos_margin}" soft_upper_limit="${2.0 * pi - safety_pos_margin}" k_position="${safety_k_position}" k_velocity="0.0"/>
-        </xacro:if>
-      </xacro:unless>
-      <xacro:if value="${joint_limited}">
-        <limit lower="${wrist_3_lower_limit}" upper="${wrist_3_upper_limit}" effort="54.0" velocity="3.2"/>
-        <xacro:if value="${safety_limits}">
-          <safety_controller soft_lower_limit="${wrist_3_lower_limit + safety_pos_margin}" soft_upper_limit="${wrist_3_upper_limit - safety_pos_margin}" k_position="${safety_k_position}" k_velocity="0.0"/>
-        </xacro:if>
-      </xacro:if>
+      <limit lower="${-1.6}" upper="${0}" effort="54.0" velocity="3.2"/>
       <dynamics damping="0.0" friction="0.0"/>
     </joint>
@@ -706,16 +662,5 @@
       <origin xyz="0.07358 0.01 -0.01452" rpy="${pi} ${pi} 0" />
       <axis xyz="0 1 0" />
-      <xacro:unless value="${joint_limited}">
-        <limit lower="${-2.0 * pi}" upper="${2.0 * pi}" effort="54.0" velocity="3.2"/>
-        <xacro:if value="${safety_limits}">
-          <safety_controller soft_lower_limit="${-2.0 * pi + safety_pos_margin}" soft_upper_limit="${2.0 * pi - safety_pos_margin}" k_position="${safety_k_position}" k_velocity="0.0"/>
-        </xacro:if>
-      </xacro:unless>
-      <xacro:if value="${joint_limited}">
-        <limit lower="${wrist_3_lower_limit}" upper="${wrist_3_upper_limit}" effort="54.0" velocity="3.2"/>
-        <xacro:if value="${safety_limits}">
-          <safety_controller soft_lower_limit="${wrist_3_lower_limit + safety_pos_margin}" soft_upper_limit="${wrist_3_upper_limit - safety_pos_margin}" k_position="${safety_k_position}" k_velocity="0.0"/>
-        </xacro:if>
-      </xacro:if>
+      <limit lower="${0}" upper="${1.6}" effort="54.0" velocity="3.2"/>
       <dynamics damping="0.0" friction="0.0"/>
     </joint>
@@ -745,16 +690,5 @@
       <origin xyz="-0.07358 -0.01 -0.01452" rpy="${pi} ${pi} ${pi}" />
       <axis xyz="0 1 0" />
-      <xacro:unless value="${joint_limited}">
-        <limit lower="${-2.0 * pi}" upper="${2.0 * pi}" effort="54.0" velocity="3.2"/>
-        <xacro:if value="${safety_limits}">
-          <safety_controller soft_lower_limit="${-2.0 * pi + safety_pos_margin}" soft_upper_limit="${2.0 * pi - safety_pos_margin}" k_position="${safety_k_position}" k_velocity="0.0"/>
-        </xacro:if>
-      </xacro:unless>
-      <xacro:if value="${joint_limited}">
-        <limit lower="${wrist_3_lower_limit}" upper="${wrist_3_upper_limit}" effort="54.0" velocity="3.2"/>
-        <xacro:if value="${safety_limits}">
-          <safety_controller soft_lower_limit="${wrist_3_lower_limit + safety_pos_margin}" soft_upper_limit="${wrist_3_upper_limit - safety_pos_margin}" k_position="${safety_k_position}" k_velocity="0.0"/>
-        </xacro:if>
-      </xacro:if>
+      <limit lower="${0}" upper="${1.6}" effort="54.0" velocity="3.2"/>
       <dynamics damping="0.0" friction="0.0"/>
     </joint>
@@ -779,4 +713,32 @@
       </inertial>
     </link>
+    <gazebo>
+ 	 <plugin name="mimic" filename="libroboticsgroup_gazebo_mimic_joint_plugin.so">
+	    <joint>${prefix}leftTilted_link</joint>
+	    <mimicJoint>${prefix}leftStraight_link</mimicJoint>
+            <multiplier>1</multiplier>
+	 </plugin>
+    </gazebo>
+    <gazebo>
+ 	 <plugin name="mimic2" filename="libroboticsgroup_gazebo_mimic_joint_plugin.so">
+	    <joint>${prefix}rightTilted_link</joint>
+	    <mimicJoint>${prefix}rightStraight_link</mimicJoint>
+            <multiplier>1</multiplier>
+	 </plugin>
+    </gazebo>
+    <gazebo>
+ 	 <plugin name="mimic3" filename="libroboticsgroup_gazebo_mimic_joint_plugin.so">
+	    <joint>${prefix}leftTilted_link</joint>
+	    <mimicJoint>${prefix}left_finger</mimicJoint>
+            <multiplier>-1</multiplier>
+	 </plugin>
+    </gazebo>
+    <gazebo>
+ 	 <plugin name="mimic4" filename="libroboticsgroup_gazebo_mimic_joint_plugin.so">
+	    <joint>${prefix}rightTilted_link</joint>
+	    <mimicJoint>${prefix}right_finger</mimicJoint>
+            <multiplier>1</multiplier>
+	 </plugin>
+    </gazebo>
     <link name="sonar_link">
       <collision>

Commit message: fixed error in suii.xacro

File: Suii/suii_description/urdf/suii.xacro (robot description, xacro)
@@ -35,7 +35,7 @@
     <xacro:property name="wheel_mass" value="0.37904"/>
     <xacro:property name="gripper_base_mass" value="0.500"/>
-    <xacro:property name="Tilted_link" value="0.035"/>
-    <!-- <xacro:property name="" value="0.500"/>
-    <xacro:property name="" value="0.500"/> -->
+    <xacro:property name="Tilted_link_mass" value="0.035"/>
+    <xacro:property name="straight_link_mass" value="0.042"/>
+    <xacro:property name="finger_mass" value="0.035"/>
     <xacro:property name="shoulder_cog" value="0.0 -0.02 0.0" />
     <xacro:property name="upper_arm_cog" value="0.13 0.0 0.1157" />
@@ -259,5 +259,5 @@
       </xacro:unless>
       <xacro:if value="${joint_limited}">
-        <limit lower="${ur3_mount_lower_limit}" upper="${ur3_mount_upper_limit}" effort="330.0" velocity="2.16"/>
+        <limit lower="${shoulder_pan_lower_limit}" upper="${shoulder_pan_upper_limit}" effort="330.0" velocity="2.16"/>
         <xacro:if value="${safety_limits}">
           <safety_controller soft_lower_limit="${ur3_mount_lower_limit + safety_pos_margin}" soft_upper_limit="${ur3_mount_upper_limit - safety_pos_margin}" k_position="${safety_k_position}" k_velocity="0.0"/>
@@ -637,5 +637,5 @@
       <dynamics damping="0.0" friction="0.0"/>
     </joint>
-    <link name="${prefix}lefStraight_link">
+    <link name="${prefix}leftStraight_link">
       <visual>
         <geometry>

Commit message: fixed inertial error gripper

File: Suii/suii_description/urdf/suii.xacro (robot description, xacro)
@@ -508,6 +508,6 @@
     <joint name="${prefix}wrist_3_link" type="revolute">
       <parent link="${prefix}wrist_3_link" />
-      <child link = "${prefix}gripper_base" />1.4771E-10
-      <origin xyz="0 0.08 0" rpy="0 1.57 -1.57" />
+      <child link = "${prefix}gripper_base"/>
+      <origin xyz="0 0.085 0" rpy="0 1.57 -1.57" />
       <axis xyz="0 1 0" />
       <xacro:unless value="${joint_limited}">
@@ -541,5 +541,6 @@
       <inertial>
         <mass value= "${gripper_base_mass}"/>
-        <inertia ixx="3.1166E-10" ixy="-4.678E-12" ixz="1.861E-11" iyy="8.724E-10" iyz="5.6254E-11" izz="6.5089E-10"/>
+        <!-- <inertia ixx="3.1166E-10" ixy="-4.678E-12" ixz="1.861E-11" iyy="8.724E-10" iyz="5.6254E-11" izz="6.5089E-10"/>  -->
+        <inertia ixx="0" ixy="0" ixz="0" iyy="0" iyz="0" izz="0"/>
         <origin xyz="0 0 0"  rpy="0 0 0" />
       </inertial>

Commit message: Sensor Updates + Tests

File: Suii/suii_description/urdf/suii.xacro (robot description, xacro)
@@ -861,4 +861,54 @@
       <child link="hokuyo_link_front"/>
     </joint>
+    <!-- Camera -->
+    <joint name="${prefix}camera_joint" type="fixed">
+      <axis xyz="0 1 0" />
+      <origin xyz="0.0 0.1 0.045" rpy="0 0 ${pi/2}"/>
+      <parent link="${prefix}gripper_base"/>
+      <child link="${prefix}camera_link"/>
+    </joint>
+    <link name="${prefix}camera_link">
+      <collision>
+        <origin xyz="0 0 0" rpy="0 0 0"/>
+        <geometry>
+           <box size="0.010 0.121 0.018"/>
+        </geometry>
+      </collision>
+      <visual>
+        <geometry>
+  	       <box size="0.010 0.121 0.018"/>
+        </geometry>
+        <material name="red">
+          <color rgba="0.8 0.0 0.0 1.0"/>
+        </material>
+      </visual>
+      <inertial>
+        <mass value="1e-5" />
+        <origin xyz="0 0 0" rpy="0 0 0"/>
+        <inertia ixx="0" ixy="0" ixz="0" iyy="0" iyz="0" izz="0" />
+      </inertial>
+    </link>
+    <!-- generate an optical frame http://www.ros.org/reps/rep-0103.html#suffix-frames
+        so that ros and opencv can operate on the camera frame correctly -->
+    <joint name="${prefix}camera_optical_joint_2D" type="fixed">
+      <!-- these values have to be these values otherwise the gazebo camera image
+          won't be aligned properly with the frame it is supposedly originating from -->
+      <axis xyz="0 1 0" />
+      <origin xyz="0 0 0" rpy="0 0 0"/>
+      <parent link="${prefix}camera_link"/>
+      <child link="${prefix}camera_link_optical_2D"/>
+    </joint>
+    <joint name="${prefix}camera_optical_joint_3D" type="fixed">
+      <!-- these values have to be these values otherwise the gazebo camera image
+          won't be aligned properly with the frame it is supposedly originating from -->
+      <axis xyz="0 1 0" />
+      <origin xyz="0 0 0" rpy="0 0 0"/>
+      <parent link="${prefix}camera_link"/>
+      <child link="${prefix}camera_link_optical_3D"/>
+    </joint>
+    <link name="${prefix}camera_link_optical_2D">
+    </link>
+    <link name="${prefix}camera_link_optical_3D">
+    </link>
     <xacro:suii_transmission prefix="${prefix}" hw_interface="${transmission_hw_interface}" />
     <xacro:suii_gazebo prefix="${prefix}" />

File: Suii/suii_description/urdf/suii_gazebo.xacro (robot description, xacro)
@@ -103,5 +103,5 @@
             <horizontal>
               <samples>1080</samples>
-              <resolution>0.25</resolution>
+              <resolution>1</resolution>
               <min_angle>-2.35619449</min_angle>
               <max_angle>2.35619449</max_angle>
@@ -135,5 +135,5 @@
             <horizontal>
               <samples>1080</samples>
-              <resolution>0.25</resolution>
+              <resolution>1</resolution>
               <min_angle>-2.35619449</min_angle>
               <max_angle>2.35619449</max_angle>
@@ -195,4 +195,103 @@
       </sensor>
     </gazebo>
+    <!--camera-->
+    <gazebo reference="camera_link">
+      <mu1>0.2</mu1>
+      <mu2>0.2</mu2>
+      <material>Gazebo/Red</material>
+    </gazebo>
+    <gazebo reference="camera_link">
+      <sensor name="camera_3D" type="depth">
+        <update_rate>60</update_rate>
+        <camera>
+          <horizontal_fov>1.48353</horizontal_fov>
+          <image>
+            <width>640</width>
+            <height>480</height>
+            <format>B8G8R8</format>
+          </image>
+          <clip>
+            <near>0.1</near>
+            <far>5</far>
+          </clip>
+          <noise>
+            <type>gaussian</type>
+            <mean>0.0</mean>
+            <stddev>0.007</stddev>
+          </noise>
+        </camera>
+        <plugin name="camera_controller_3D" filename="libgazebo_ros_openni_kinect.so">
+          <baseline>0.2</baseline>
+          <alwaysOn>true</alwaysOn>
+          <updateRate>1.0</updateRate>
+          <cameraName>camera_3D</cameraName>
+          <imageTopicName>/camera_3D/color/image_raw</imageTopicName>
+          <cameraInfoTopicName>/camera_3D/color/camera_info</cameraInfoTopicName>
+          <depthImageTopicName>/camera_3D/depth/image_raw</depthImageTopicName>
+          <depthImageInfoTopicName>/camera_3D/depth/camera_info</depthImageInfoTopicName>
+          <pointCloudTopicName>/camera_3D/depth/points</pointCloudTopicName>
+          <frameName>camera_link_optical_3D</frameName>
+          <pointCloudCutoff>0.2</pointCloudCutoff>
+          <pointCloudCutoffMax>1.5</pointCloudCutoffMax>
+          <distortionK1>0.00000001</distortionK1>
+          <distortionK2>0.00000001</distortionK2>
+          <distortionK3>0.00000001</distortionK3>
+          <distortionT1>0.00000001</distortionT1>
+          <distortionT2>0.00000001</distortionT2>
+          <CxPrime>0</CxPrime>
+          <Cx>0</Cx>
+          <Cy>0</Cy>
+          <focalLength>0</focalLength>
+          <hackBaseline>0</hackBaseline>
+        </plugin>
+      </sensor>
+    </gazebo>
+    <!-- camera -->
+    <gazebo reference="camera_link">
+      <sensor type="camera" name="camera_2D">
+        <update_rate>30.0</update_rate>
+        <camera name="head">
+          <horizontal_fov>1.34390352</horizontal_fov>
+          <image>
+            <width>1920</width>
+            <height>1080</height>
+            <format>R8G8B8</format>
+          </image>
+          <clip>
+            <near>0.02</near>
+            <far>300</far>
+          </clip>
+          <noise>
+            <type>gaussian</type>
+            <!-- Noise is sampled independently per pixel on each frame.
+                 That pixel's noise value is added to each of its color
+                 channels, which at that point lie in the range [0,1]. -->
+            <mean>0.0</mean>
+            <stddev>0.007</stddev>
+          </noise>
+        </camera>
+        <plugin name="camera_controller_2D" filename="libgazebo_ros_camera.so">
+          <alwaysOn>true</alwaysOn>
+          <updateRate>0.0</updateRate>
+          <cameraName>camera_2D</cameraName>
+          <imageTopicName>/camera_2D/image_raw</imageTopicName>
+          <cameraInfoTopicName>/camera_2D/camera_info</cameraInfoTopicName>
+          <frameName>camera_link_optical_2D</frameName>
+          <!-- setting hackBaseline to anything but 0.0 will cause a misalignment
+              between the gazebo sensor image and the frame it is supposed to
+              be attached to -->
+          <hackBaseline>0.0</hackBaseline>
+          <distortionK1>0.0</distortionK1>
+          <distortionK2>0.0</distortionK2>
+          <distortionK3>0.0</distortionK3>
+          <distortionT1>0.0</distortionT1>
+          <distortionT2>0.0</distortionT2>
+          <CxPrime>0</CxPrime>
+          <Cx>0.0</Cx>
+          <Cy>0.0</Cy>
+          <focalLength>0.0</focalLength>
+        </plugin>
+      </sensor>
+    </gazebo>
   </xacro:macro>
 </robot>

Commit message: removed boxes from lidar

File: Suii/suii_description/urdf/suii.xacro (robot description, xacro)
@@ -64,5 +64,5 @@
     <!-- sensor properties-->
     <xacro:property name="sonar_link" value="-0.05" /> <!-- Size of square 'sonar' box -->
-    <xacro:property name="laser_link" value="-0.05" /> <!-- Size of square 'sonar' box -->
+    <xacro:property name="laser_link" value="-0.001" /> <!-- Size of square 'sonar' box -->
     <xacro:property name="height" value="0.3" /> <!-- height sensors-->
     <xacro:property name="axel_offset" value="0.05" /> <!-- offset placement -->
@@ -766,5 +766,5 @@
         <origin xyz="0 0 0" rpy="0 0 0"/>
         <geometry>
-          <box size="0.1 0.1 0.1"/>
+          <box size="0.01 0.01 0.01"/>
         </geometry>
       </collision>
@@ -794,5 +794,5 @@
         <origin xyz="0 0 0" rpy="0 0 0"/>
         <geometry>
-          <box size="0.1 0.1 0.1"/>
+          <box size="0.01 0.01 0.01"/>
         </geometry>
       </collision>

Commit message: fixed gripper

File: Suii/suii_description/urdf/suii.xacro (robot description, xacro)
@@ -506,10 +506,10 @@
       </xacro:cylinder_inertial>
     </link>
-    <joint name="${prefix}wrist_3_link" type="revolute">
+    <joint name="${prefix}wrist_3_link" type="fixed">
       <parent link="${prefix}wrist_3_link" />
       <child link = "${prefix}gripper_base"/>
-      <origin xyz="0 0.085 0" rpy="0 1.57 -1.57" />
-      <axis xyz="0 1 0" />
-      <xacro:unless value="${joint_limited}">
+      <origin xyz="0 0.08 0" rpy="0 1.57 -1.57" />
+      <axis xyz="0 1 0" />
+      <!-- <xacro:unless value="${joint_limited}">
         <limit lower="${-2.0 * pi}" upper="${2.0 * pi}" effort="54.0" velocity="3.2"/>
         <xacro:if value="${safety_limits}">
@@ -523,5 +523,5 @@
         </xacro:if>
       </xacro:if>
-      <dynamics damping="0.0" friction="0.0"/>
+      <dynamics damping="0.0" friction="0.0"/> -->
     </joint>
     <link name="${prefix}gripper_base">
@@ -546,5 +546,5 @@
       </inertial>
     </link>
-    <joint name="${prefix}leftTilted_link" type="revolute">
+    <joint name="${prefix}leftTilted_link" type="fixed">
       <parent link="${prefix}gripper_base" />
       <child link = "${prefix}leftTilted_link" />

Commit message: Camera and Lidar fixed

File: Suii/suii_description/urdf/suii.xacro (robot description, xacro)
@@ -786,5 +786,5 @@
     <joint name="hokuyo_joint_back" type="fixed">
       <axis xyz="0 1 0" />
-      <origin xyz="0.244 0.168 0.15" rpy="0 0 ${pi/4}"/>
+      <origin xyz="0.240 0.171 0.18" rpy="0 0 ${pi/4}"/>
       <parent link="${prefix}base_link"/>
       <child link="hokuyo_link_back"/>
@@ -814,5 +814,5 @@
     <joint name="hokuyo_joint_front" type="fixed">
       <axis xyz="0 1 0" />
-      <origin xyz="-0.251153588295 -0.17189989984 0.16" rpy="0 0 ${pi/4 + pi}"/>
+      <origin xyz="-0.240 -0.171 0.18" rpy="0 0 ${pi/4 + pi}"/>
       <parent link="${prefix}base_link"/>
       <child link="hokuyo_link_front"/>
@@ -821,5 +821,5 @@
     <joint name="${prefix}camera_joint" type="fixed">
       <axis xyz="0 1 0" />
-      <origin xyz="0.0 0.1 0.045" rpy="0 0 ${pi/2}"/>
+      <origin xyz="0.0 -0.045 -0.1" rpy="0 ${pi/2} ${-pi/2}"/>
       <parent link="${prefix}gripper_base"/>
       <child link="${prefix}camera_link"/>
