Commit message: I have added the demo and changed the limits of two joints of the arm

File: Suii/suii_description/urdf/suii.xacro (robot description, xacro)
@@ -290,7 +290,7 @@
       <axis xyz="0 0 1" />
       <xacro:unless value="${joint_limited}">
-        <limit lower="${-2.0 * pi}" upper="${2.0 * pi}" effort="330.0" velocity="2.16"/>
-        <xacro:if value="${safety_limits}">
-          <safety_controller soft_lower_limit="${-2.0 * pi + safety_pos_margin}" soft_upper_limit="${2.0 * pi - safety_pos_margin}" k_position="${safety_k_position}" k_velocity="0.0"/>
+        <limit lower="${-3.0 * pi}" upper="${1.0 * pi}" effort="330.0" velocity="2.16"/>
+        <xacro:if value="${safety_limits}">
+          <safety_controller soft_lower_limit="${-3.0 * pi + safety_pos_margin}" soft_upper_limit="${1.0 * pi - safety_pos_margin}" k_position="${safety_k_position}" k_velocity="0.0"/>
         </xacro:if>
       </xacro:unless>
@@ -327,7 +327,7 @@
       <axis xyz="0 1 0" />
       <xacro:unless value="${joint_limited}">
-        <limit lower="${-2.0 * pi}" upper="${2.0 * pi}" effort="330.0" velocity="2.16"/>
-        <xacro:if value="${safety_limits}">
-          <safety_controller soft_lower_limit="${-2.0 * pi + safety_pos_margin}" soft_upper_limit="${2.0 * pi - safety_pos_margin}" k_position="${safety_k_position}" k_velocity="0.0"/>
+        <limit lower="${-2.5 * pi}" upper="${1.5 * pi}" effort="330.0" velocity="2.16"/>
+        <xacro:if value="${safety_limits}">
+          <safety_controller soft_lower_limit="${-2.5 * pi + safety_pos_margin}" soft_upper_limit="${1.5 * pi - safety_pos_margin}" k_position="${safety_k_position}" k_velocity="0.0"/>
         </xacro:if>
       </xacro:unless>

Commit message: latest

File: Suii/suii_description/urdf/suii.xacro (robot description, xacro)
@@ -546,5 +546,5 @@
       </inertial>
     </link>
-    <joint name="${prefix}leftTilted_link" type="fixed">
+    <joint name="${prefix}leftTilted_link" type="revolute">
       <parent link="${prefix}gripper_base" />
       <child link = "${prefix}leftTilted_link" />
